File: pcb/RCPlaneShield/RCPlaneShield.kicad_pcb (KiCad board)
At the start: 2 copper layers, 102.4 x 53.3 mm, 32 parts, among them J1 Roll-D12, J10 Batt Meas-A0, J11 NavLed-D13, J12 NRF24L01 Direct, J13 NRF24L01, J2 Pitch-D11, J3 Yaw-D10, J4 Flaps-D9, J5 Nose Gear-D8, J6 L-Gear-D7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

Commit message: Update pcb to v1.1 - wider servo traces, BEC drives servos
Parts:
- added D2: Servo Pwr, LED_THT:LED_D5.0mm, F.Cu at (134.7, 113.9)
- added J14: BEC Jmpr, Connector_PinHeader_2.54mm:PinHeader_1x02_P2.54mm_Vertical, F.Cu at (160.0, 96.5)
- added R5: 330, Resistor_THT:R_Axial_DIN0309_L9.0mm_D3.2mm_P12.70mm_Horizontal, F.Cu at (149.9, 101.6)
- D1: value Power LED -> Ard 5V Pwr
- J1: value Roll-D12 -> L-Roll-D12
- J2: value Pitch-D11 -> R-Roll-D11
- J3: value Yaw-D10 -> L-Pitch-D10
- J4: value Flaps-D9 -> R-Pitch-D9
- R1: value 3M -> 4.7M
- R2: value 1M -> 1.5M
- R3, R4: value 300 -> 330
- SW1: value MODE-D0 -> SW_SPDT; footprint Button_Switch_THT:SW_DIP_SPSTx01_Slide_9.78x4.72mm_W7.62mm_P2.54mm -> Button_Switch_THT:SW_Slide_1P2T_CK_OS102011MS2Q
- moved R2 5.08 mm to (154.9, 101.6)
- moved R1 2.54 mm to (160.0, 101.6)
- moved SW1 1.23 mm to (182.9, 78.7)
Connections:
- J1 pad 2: +5V -> Net-(J14-Pad2)
- J2 pad 2: +5V -> Net-(J14-Pad2)
- J3 pad 2: +5V -> Net-(J14-Pad2)
- J4 pad 2: +5V -> Net-(J14-Pad2)
- J5 pad 2: +5V -> Net-(J14-Pad2)
- J6 pad 2: +5V -> Net-(J14-Pad2)
- J7 pad 2: +5V -> Net-(J14-Pad2)
- J8 pad 2: /Vin -> Net-(J14-Pad2)
Routing:
- net Net-(J14-Pad2): track 0.00 -> 184.7 mm
- net +5V: track 262.9 -> 133.9 mm, vias 3 -> 2
- net /Vin: track 36.9 -> 0.00 mm, vias 2 -> 0
- net Net-(D2-Pad1): track 0.00 -> 20.3 mm
- net /5(**): track 83.3 -> 93.4 mm
- net GND: track 315.9 -> 322.5 mm
- net /4(**): track 74.6 -> 80.6 mm
- net /0(Rx0): track 18.0 -> 20.1 mm
- net /8(**): track 18.9 -> 16.9 mm
- net /3(**): track 117.8 -> 116.8 mm
- net Net-(J10-Pad1): track 10.8 -> 9.72 mm
- net /51(MOSI): track 34.1 -> 34.7 mm
- net /A0: track 22.1 -> 22.6 mm
Other:
- board text added: "1.5M"
- board text added: "330"
- board text added: "4.7M"
- board text added: "Arduino Pwr"
- board text added: "BEC/5V Jmpr"
- board text added: "Batt Meas-A0"
- board text added: "CE"
- board text added: "FRHS RC Plane Interface v1.1"
- board text added: "LPitch-D10"
- board text added: "LRoll-D12"
- board text added: "RPitch-D9"
- board text added: "RRoll-D11"
- board text added: "Servo Pwr"
- board text removed: "1M"
- board text removed: "300"
- board text removed: "3M"
- board text removed: "Batt-Meas-A0"
- board text removed: "FRHS RC Plane Interface v1.0"
- board text removed: "Flaps-D9"
- board text removed: "Pitch-D11"
- board text removed: "Power"
- board text removed: "Roll-D12"
- board text removed: "Yaw-D10"
